File: hardware/detector.sch (EAGLE design)
At the start: 40 parts, among them J2 AVR_SPI_PRG_6NS, Q2 16MHz, T1 BC337, T3 BC337, U2 TINY85-20-DIP

Commit message: hardware: separate DIP and SIL drawings for mega328p, gitignore tuning
Parts:
- removed C10, C9: 22p, resistor:C-EU050-024X044
- removed D6: G, SparkFun-LED:LED3MM
- removed D7: Y, SparkFun-LED:LED3MM
- removed JP6: (no value), jumper:JP2E
- removed R12: 4k7, resistor:R-EU_0204/5
- removed R13: 1k, resistor:R-EU_0204/5
- added C5, C6: 1u, capacitor-wima:C-2.5-5/4
- added D1, D2: 24V, SparkFun-DiscreteSemi:DIODE-ZENER
- added JP4: (no value), jumper:JP3QE
- added R2: 470, resistor:R-EU_0204/5
- added R3: 75, resistor:R-EU_0204/7
- C7, C8: value 1u -> 22p; device capacitor-wima:C-2.5-5/4 -> resistor:C-EU050-024X044
- D3: value 24V -> R; device SparkFun-DiscreteSemi:DIODE-ZENER -> SparkFun-LED:LED3MM
- D4: value 24V -> G; device SparkFun-DiscreteSemi:DIODE-ZENER -> SparkFun-LED:LED3MM
- D5: value R -> Y
- JP5: device jumper:JP3QE -> jumper:JP2E
- R1: value 75 -> 1M8; device resistor:R-EU_0204/7 -> resistor:R-EU_0204/5
- R4: value 1k -> 4k7
- R5: value 470 -> 1k
- R6: value 4k7 -> 1k
- R9: value 1M8 -> 4k7
- renumbered F1 to Q1, J2 to J1, R14 to R7, R15 to R8, R16 to R11, T3 to T2, U2 to U1
Connections:
- net FREQ: now also R5.1; no longer R4.1
- net GND: now also C5.2, C6.1, C6.2, C7.1, D5.C, JP4-1.2, JP4-2.2, JP4-3.1, JP5.3, R6.2; no longer C10.1, C7.2, C8.2, C9.1, D7.C, JP5-1.2, JP5-2.2, JP5-3.1, JP6.3, R10.2
- net GND-ISO: now also GDT1.1, R1.1; no longer GDT2.1, R9.1
- net N$1: now also D1.C, D2.C; no longer D3.C, D4.C
- net N$14: now also D1.A, R3.1, R4.2; no longer D3.A, R1.1, R6.2
- net N$2: now also R4.1; no longer R6.1
- net N$20: now also R9.1; no longer R12.1
- net N$21: now also GDT1.2, GDT2.1, R1.2; no longer GDT1.1, GDT2.2, R9.2
- net N$22: now also D3.C, R6.1; no longer D5.C, R10.1
- net N$23: now also D4.C, JP5.2; no longer D6.C, JP6.2
- net N$24: now also D4.A; no longer D6.A
- net N$25: now also C7.2; no longer C10.2
- net N$26: now also C8.2; no longer C9.2
- net N$27: now also D5.A, R10.2; no longer D7.A, R13.2
- net N$28: now also R10.1; no longer R13.1
- net N$29: now also R9.2; no longer R12.2
- net N$3: now also R2.1; no longer R5.1
- net N$6: now also D2.A, R2.2; no longer D4.A, R5.2
- net N$7: now also GDT2.2; no longer GDT1.2
- net VCC: now also C5.1, D3.A, JP4-1.1, JP4-2.1, JP4-3.2, JP5.1, R3.2, R5.2; no longer C7.1, D5.A, JP5-1.1, JP5-2.1, JP5-3.2, JP6.1, R1.2, R4.2
