File: hardware/detector_t85-pu.brd (EAGLE design)
At the start: 84.8 x 48.2 mm, 40 parts, among them J1 AVR_SPI_PRG_6NS, Q1 BS170, Q2 16MHz, T1 BC337, T2 BC337, U1 TINY85-20-DIP

Commit message: hardware: t85 board fuckery
Parts:
- added C9: 1u, rcl:C050-025X075
- C5, C6: device capacitor-wima:C2.5/5-4 -> rcl:C050-025X075
- Q1: value BS170 -> BS170.; device transistor-small-signal:SOT54E -> detector:TO92-DGS
- moved X1 46.7 mm to (38.1, 44.5), turned to 0 degrees
- moved GDT2 32.4 mm to (38.1, 33.0), turned to 180 degrees
- moved R1 22.9 mm to (40.6, 26.7), turned to 0 degrees
- moved GDT1 17.1 mm to (39.4, 20.3), turned to 0 degrees
- moved D1 8.98 mm to (45.7, 12.7), turned to 90 degrees
- moved C8 4.02 mm to (50.8, 25.4), turned to 270 degrees
- moved C7 3.81 mm to (50.8, 27.9)
- moved R2 2.84 mm to (58.4, 19.1)
- moved C6 1.27 mm to (73.7, 40.6), turned to 0 degrees
- moved C5 1.27 mm to (71.1, 6.35)
- moved L1 1.27 mm to (38.1, 6.35)
- moved C1 1.27 mm to (48.3, 5.08)
- moved C2 1.27 mm to (50.8, 5.08)
- moved C3 1.27 mm to (53.3, 5.08)
- moved C4 1.27 mm to (55.9, 5.08)
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Connections:
- net GND: now also C9.2; no longer C6.1
- net GND-ISO: now also X1.2; no longer X1.3
- net N$21: now also L1.6, X1.3; no longer L1.4, X1.2
- net N$7: now also L1.4; no longer L1.6
- net VCC: now also C6.1, C9.1
Other:
- board size 84.8 x 48.2 mm -> 54.3 x 48.2 mm

Commit message: hardware-t85: almost there
Parts:
- moved D5 31.4 mm to (49.5, 41.9)
- moved R10 10.5 mm to (53.3, 40.6), turned to 90 degrees
- moved R11 2.84 mm to (62.2, 38.1), turned to 0 degrees
- moved C9 2.54 mm to (64.8, 19.1), turned to 180 degrees
- moved J1 2.54 mm to (61.0, 43.2)
- moved U1 2.54 mm to (62.2, 27.9)
- moved T2 2.01 mm to (73.0, 37.5)
- moved Q2 1.27 mm to (54.6, 26.7)
- moved R2 1.27 mm to (57.1, 19.1)
- moved C7 1.27 mm to (49.5, 27.9)
- moved C8 1.27 mm to (49.5, 25.4)
- moved R9 1.27 mm to (72.4, 30.5)
Routing:
- net GND: track 0.00 -> 111.7 mm
- net VCC: track 0.00 -> 90.8 mm, vias 0 -> 8
- net N$21: track 0.00 -> 45.9 mm
- net N$7: track 0.00 -> 36.2 mm
- net N$14: track 0.00 -> 26.3 mm
- net GND-ISO: track 0.00 -> 25.1 mm
- net N$2: track 0.00 -> 21.4 mm
- net N$6: track 0.00 -> 20.8 mm
- net N$30: track 0.00 -> 6.88 mm
- net FREQ: track 0.00 -> 6.35 mm
- net N$5: track 0.00 -> 3.81 mm
- net N$4: track 0.00 -> 3.81 mm
- net N$11: track 0.00 -> 3.81 mm

Commit message: hardware-t85: really almost there
Parts:
- D1, D2: device SparkFun-DiscreteSemi:DIODE-BZT52 -> diode:ZDIO-5
- moved D5 31.4 mm to (80.0, 34.3), turned to 90 degrees
- moved R10 21.7 mm to (73.7, 33.0), turned to 0 degrees
- moved R6 9.25 mm to (73.7, 21.6), turned to 180 degrees
- moved R7 2.54 mm to (73.7, 25.4), turned to 180 degrees
- moved R9 1.80 mm to (73.7, 29.2), turned to 180 degrees
- moved R5 1.27 mm to (64.8, 14.0)
- moved D1 1.27 mm to (47.0, 12.7), turned to 270 degrees
- moved D2 1.27 mm to (53.3, 16.5), turned to 0 degrees
- moved C7 1.27 mm to (49.5, 29.2)
- moved Q2 1.27 mm to (54.6, 27.9)
- moved R2 1.27 mm to (55.9, 19.1)
- moved R8 1.27 mm to (67.3, 14.0)
- moved R3 0.90 mm to (60.3, 13.3)
Routing:
- net GND: track 111.7 -> 198.3 mm
- net N$31: track 0.00 -> 58.2 mm
- net VCC: track 90.8 -> 137.6 mm
- net N$28: track 0.00 -> 33.6 mm
- net N$29: track 0.00 -> 29.9 mm
- net N$23: track 0.00 -> 19.9 mm
- net N$3: track 0.00 -> 17.9 mm
- net N$26: track 0.00 -> 10.5 mm
- net N$25: track 0.00 -> 9.94 mm
- net N$20: track 0.00 -> 9.57 mm
- net N$30: track 6.88 -> 12.3 mm
- net N$24: track 0.00 -> 4.34 mm
- net N$22: track 0.00 -> 4.34 mm
- net N$1: track 0.00 -> 4.34 mm
- net N$27: track 0.00 -> 3.81 mm
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