File: hardware/detector328p-au.sch (EAGLE design)
At the start: 65 parts, among them K1 SRD-05VDC-SL-C, Q1 BSS123, Q2 16MHz, T1 BC817-40SMD, T2 BC817, T3 BC817, U1 ATMEGA328P-AU

Commit message: detector328p-au serial port
Parts:
- added SERIAL: (no value), con-lstb:MA03-1
Connections:
- new net N$39: SERIAL.1, U1.PD0
- new net N$48: SERIAL.3, U1.PD1
- net GND: now also SERIAL.2
Changed lines of the file:
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@@
 <part name="LCD" library="con-lstb" deviceset="MA04-1" device=""/>
 <part name="POWER" library="con-lstb" deviceset="MA03-2" device=""/>
+<part name="SERIAL" library="con-lstb" deviceset="MA03-1" device=""/>
 </parts>
 <sheets>
@@
 <instance part="OUT" gate="G$1" x="-2.54" y="38.1" rot="MR180"/>
 <instance part="LCD" gate="1" x="198.12" y="66.04" rot="R180"/>
+<instance part="SERIAL" gate="G$1" x="198.12" y="53.34" rot="R180"/>
 </instances>
 <busses>
@@
 <segment>
 <pinref part="GND25" gate="1" pin="GND"/>
-<wire x1="185.42" y1="12.7" x2="185.42" y2="71.12" width="0.1524" layer="91"/>
+<wire x1="185.42" y1="12.7" x2="185.42" y2="53.34" width="0.1524" layer="91"/>
+<wire x1="185.42" y1="53.34" x2="185.42" y2="71.12" width="0.1524" layer="91"/>
 <wire x1="185.42" y1="71.12" x2="190.5" y2="71.12" width="0.1524" layer="91"/>
 <wire x1="154.94" y1="88.9" x2="185.42" y2="88.9" width="0.1524" layer="91"/>
@@
 <pinref part="RESET" gate="1" pin="S"/>
 <pinref part="LCD" gate="1" pin="1"/>
+<pinref part="SERIAL" gate="G$1" pin="2"/>
+<wire x1="190.5" y1="53.34" x2="185.42" y2="53.34" width="0.1524" layer="91"/>
+<junction x="185.42" y="53.34"/>
 </segment>
 </net>
@@
 <segment>
 <pinref part="R16" gate="G$1" pin="1"/>
-<wire x1="152.4" y1="45.72" x2="195.58" y2="45.72" width="0.1524" layer="91"/>
-<label x="187.198" y="46.228" size="1.778" layer="95"/>
+<wire x1="152.4" y1="45.72" x2="160.02" y2="45.72" width="0.1524" layer="91"/>
+<wire x1="160.02" y1="45.72" x2="160.02" y2="38.1" width="0.1524" layer="91"/>
+<wire x1="160.02" y1="38.1" x2="195.58" y2="38.1" width="0.1524" layer="91"/>
+<label x="189.738" y="38.608" size="1.778" layer="95"/>
 </segment>
 </net>
@@
 </segment>
 </net>
+<net name="N$39" class="0">
+<segment>
+<pinref part="U1" gate="A" pin="PD0"/>
+<pinref part="SERIAL" gate="G$1" pin="1"/>
+<wire x1="137.16" y1="55.88" x2="190.5" y2="55.88" width="0.1524" layer="91"/>
+</segment>
+</net>
+<net name="N$48" class="0">
+<segment>
+<pinref part="SERIAL" gate="G$1" pin="3"/>
+<wire x1="190.5" y1="50.8" x2="160.02" y2="50.8" width="0.1524" layer="91"/>
+<wire x1="160.02" y1="50.8" x2="160.02" y2="53.34" width="0.1524" layer="91"/>
+<pinref part="U1" gate="A" pin="PD1"/>
+<wire x1="160.02" y1="53.34" x2="137.16" y2="53.34" width="0.1524" layer="91"/>
+</segment>
+</net>

Commit message: detector328p-au R2->1K, T1->BC817
Parts:
- R2: value 470 -> 1K
- T1: value BC817-40SMD -> BC817
Changed lines of the file:
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@@
 <parts>
 <part name="R6" library="resistor" deviceset="R-EU_" device="R0603" value="1k"/>
-<part name="R2" library="resistor" deviceset="R-EU_" device="R0603" value="470"/>
+<part name="R2" library="resistor" deviceset="R-EU_" device="R0603" value="1K"/>
 <part name="R5" library="resistor" deviceset="R-EU_" device="R0603" value="4k7"/>
 <part name="Q1" library="transistor-small-signal" deviceset="BSS123" device=""/>
@@
 <part name="GND5" library="supply1" deviceset="GND" device=""/>
 <part name="P+1" library="supply1" deviceset="VCC" device=""/>
-<part name="T1" library="transistor-npn" deviceset="BC817*" device="SMD" technology="-40" value="BC817-40SMD"/>
+<part name="T1" library="transistor-npn" deviceset="BC817*" device="SMD" technology="-40" value="BC817"/>
 <part name="GND4" library="supply1" deviceset="GND" device=""/>
 <part name="GND3" library="supply1" deviceset="GND" device=""/>
