File: hardware/eagle/detector328p-au.brd (EAGLE design)
At the start: 40 x 70 mm, 68 parts, among them K1 SRD-05VDC-SL-C, Q1 BSS123, Q2 16MHz, T1 BC817, T2 BC817, T3 BC817, U1 ATMEGA328P-AU

Commit message: detector_t85-pu: T2 10K pull-up, Zener 5,1V -> 20V
Parts:
- added R24: 10k, resistor:R0603
- D1, D2: value 5.1V 0.5W -> 20V 0.5W
- moved D4 0.51 mm to (33.0, 64.8)
- moved R8 0.36 mm to (32.0, 67.1), turned to 90 degrees
Connections:
- net N$23: now also R24.1
- net VCC: now also R24.2
Routing:
- net N$23: track 5.13 -> 7.14 mm
- net N$24: track 2.05 -> 1.49 mm
Changed lines of the file:
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@@
 <attribute name="VALUE" x="25.273" y="55.245" size="1.27" layer="27" rot="R180"/>
 </element>
-<element name="D1" library="diode" package="SOD80C" value="5.1V 0.5W" x="12.7" y="31.242" smashed="yes" rot="MR180">
+<element name="D1" library="diode" package="SOD80C" value="20V 0.5W" x="12.7" y="31.242" smashed="yes" rot="MR180">
 <attribute name="NAME" x="13.208" y="29.083" size="0.8128" layer="26" font="vector" rot="MR0"/>
 <attribute name="VALUE" x="11.176" y="33.655" size="1.27" layer="28" rot="MR180"/>
@@
 <attribute name="VALUE" x="36.068" y="34.7345" size="0.4064" layer="27"/>
 </element>
-<element name="D2" library="diode" package="SOD80C" value="5.1V 0.5W" x="6.604" y="31.242" smashed="yes" rot="MR0">
+<element name="D2" library="diode" package="SOD80C" value="20V 0.5W" x="6.604" y="31.242" smashed="yes" rot="MR0">
 <attribute name="NAME" x="7.112" y="29.083" size="0.8128" layer="26" font="vector" rot="MR0"/>
 <attribute name="VALUE" x="8.128" y="28.829" size="1.27" layer="28" rot="MR0"/>
@@
 <attribute name="VALUE" x="14.224" y="59.4995" size="0.4064" layer="27" rot="R180"/>
 </element>
-<element name="D4" library="SparkFun-LED" package="LED-0603" value="B" x="33.528" y="64.77" smashed="yes" rot="R270">
-<attribute name="NAME" x="31.877" y="63.1825" size="0.8128" layer="25" font="vector"/>
-<attribute name="VALUE" x="32.512" y="63.6905" size="0.4064" layer="27"/>
+<element name="D4" library="SparkFun-LED" package="LED-0603" value="B" x="33.02" y="64.77" smashed="yes" rot="R270">
+<attribute name="NAME" x="31.369" y="63.1825" size="0.8128" layer="25" font="vector"/>
+<attribute name="VALUE" x="32.004" y="63.6905" size="0.4064" layer="27"/>
 </element>
 <element name="D5" library="diode" package="SOD80C" value="" x="32.766" y="37.338" smashed="yes" rot="MR0">
@@
 <attribute name="VALUE" x="8.001" y="60.833" size="1.27" layer="28" rot="MR90"/>
 </element>
-<element name="R8" library="resistor" package="R0603" value="1k" x="31.75" y="66.802" smashed="yes" rot="R180">
-<attribute name="NAME" x="32.639" y="68.453" size="0.8128" layer="25" font="vector" rot="R180"/>
-<attribute name="VALUE" x="32.385" y="68.707" size="1.27" layer="27" rot="R180"/>
+<element name="R8" library="resistor" package="R0603" value="1k" x="32.004" y="67.056" smashed="yes" rot="R90">
+<attribute name="NAME" x="31.369" y="68.707" size="0.8128" layer="25" font="vector"/>
+<attribute name="VALUE" x="33.909" y="66.421" size="1.27" layer="27" rot="R90"/>
 </element>
 <element name="R9" library="resistor" package="R0603" value="4k7" x="33.782" y="45.72" smashed="yes" rot="MR90">
@@
 <attribute name="NAME" x="13.335" y="41.148" size="0.8128" layer="25" font="vector" ratio="10" rot="R270"/>
 <attribute name="VALUE" x="13.081" y="42.926" size="1.27" layer="27" ratio="10" rot="R270"/>
+</element>
+<element name="R24" library="resistor" package="R0603" value="10k" x="34.036" y="67.056" smashed="yes" rot="R90">
+<attribute name="NAME" x="33.147" y="68.707" size="0.8128" layer="25" font="vector"/>
+<attribute name="VALUE" x="35.941" y="66.421" size="1.27" layer="27" rot="R90"/>
 </element>
 </elements>
@@
 <wire x1="30.48" y1="64.096" x2="29.806" y2="64.77" width="0.508" layer="1"/>
 <wire x1="29.806" y1="64.77" x2="27.94" y2="64.77" width="0.508" layer="1"/>
-<wire x1="36.83" y1="67.31" x2="34.544" y2="67.31" width="0.508" layer="1"/>
-<wire x1="34.544" y1="67.31" x2="33.782" y2="68.072" width="0.508" layer="1"/>
-<wire x1="33.782" y1="68.072" x2="31.242" y2="68.072" width="0.508" layer="1"/>
-<wire x1="31.242" y1="68.072" x2="30.988" y2="67.818" width="0.508" layer="1"/>
-<wire x1="30.988" y1="67.818" x2="30.9" y2="67.73" width="0.508" layer="1"/>
-<wire x1="30.9" y1="67.73" x2="30.9" y2="66.802" width="0.508" layer="1"/>
 <wire x1="22.352" y1="59.69" x2="24.218" y2="61.556" width="0.508" layer="1"/>
 <wire x1="24.218" y1="61.556" x2="25.146" y2="61.556" width="0.508" layer="1"/>
-<wire x1="29.806" y1="64.77" x2="30.9" y2="65.864" width="0.508" layer="1"/>
-<wire x1="30.9" y1="65.864" x2="30.9" y2="66.802" width="0.508" layer="1"/>
 <contactref element="K1" pad="2"/>
 <contactref element="D5" pad="C"/>
@@
 <wire x1="8.128" y1="49.872" x2="10.16" y2="49.872" width="0.254" layer="1"/>
 <wire x1="10.16" y1="49.872" x2="10.326" y2="50.038" width="0.254" layer="1"/>
+<contactref element="R24" pad="2"/>
+<wire x1="29.806" y1="64.77" x2="29.806" y2="66.128" width="0.508" layer="1"/>
+<wire x1="29.806" y1="66.128" x2="29.972" y2="66.294" width="0.508" layer="1"/>
+<wire x1="29.972" y1="66.294" x2="31.584" y2="67.906" width="0.508" layer="1"/>
+<wire x1="31.584" y1="67.906" x2="32.004" y2="67.906" width="0.508" layer="1"/>
+<wire x1="32.004" y1="67.906" x2="34.036" y2="67.906" width="0.508" layer="1"/>
+<wire x1="34.036" y1="67.906" x2="34.632" y2="67.31" width="0.508" layer="1"/>
+<wire x1="34.632" y1="67.31" x2="36.83" y2="67.31" width="0.508" layer="1"/>
 </signal>
 <signal name="FREQ">
@@
 <contactref element="T2" pad="C"/>
 <contactref element="OUT" pad="2"/>
-<wire x1="34.405" y1="64.77" x2="36.83" y2="64.77" width="0.254" layer="1"/>
 <wire x1="34.12" y1="64.77" x2="36.83" y2="64.77" width="0.254" layer="16"/>
+<contactref element="R24" pad="1"/>
+<wire x1="33.897" y1="64.77" x2="33.897" y2="66.067" width="0.254" layer="1"/>
+<wire x1="33.897" y1="66.067" x2="34.036" y2="66.206" width="0.254" layer="1"/>
+<wire x1="33.897" y1="64.77" x2="36.83" y2="64.77" width="0.254" layer="1"/>
 </signal>
 <signal name="N$24">
 <contactref element="D4" pad="A"/>
 <contactref element="R8" pad="1"/>
-<wire x1="32.651" y1="64.77" x2="32.6" y2="64.821" width="0.254" layer="1"/>
-<wire x1="32.6" y1="64.821" x2="32.6" y2="66.802" width="0.254" layer="1"/>
+<wire x1="32.004" y1="66.206" x2="32.143" y2="66.067" width="0.254" layer="1"/>
+<wire x1="32.143" y1="66.067" x2="32.143" y2="64.77" width="0.254" layer="1"/>
 </signal>
 <signal name="N$27">
