File: hardware/kicad/stm32f030/ledbar.sch (KiCad schematic (older format))
At the start: 22 parts, among them U3 MCP23017

Commit message: hardware/kicad/stm32f030: modules ready
Parts:
- RN1, RN2, RN3, RN4: footprint Resistors_SMD:R_Array_Convex_4x0603 -> Resistors_SMD:R_Array_Convex_4x0603_HandSoldering
Connections:
- net at U3.21 (GPA0): now also LED3.1 (K); no longer LED10.1 (K)
- net at U3.22 (GPA1): now also LED4.1 (K); no longer LED9.1 (K)
- net at U3.23 (GPA2): now also LED5.1 (K); no longer LED8.1 (K)
- net at U3.24 (GPA3): now also LED6.1 (K); no longer LED7.1 (K)
- net at U3.25 (GPA4): now also LED7.1 (K); no longer LED6.1 (K)
- net at U3.26 (GPA5): now also LED8.1 (K); no longer LED5.1 (K)
- net at U3.27 (GPA6): now also LED9.1 (K); no longer LED4.1 (K)
- net at U3.28 (GPA7): now also LED10.1 (K); no longer LED3.1 (K)
- no-connect marks 0 -> 3
Changed lines of the file:
@@
 F 0 "RN1" V 4350 2500 50  0000 C CNN
 F 1 "330" V 4850 2500 50  0000 C CNN
-F 2 "Resistors_SMD:R_Array_Convex_4x0603" V 4925 2500 50  0001 C CNN
+F 2 "Resistors_SMD:R_Array_Convex_4x0603_HandSoldering" V 4925 2500 50  0001 C CNN
 F 3 "" H 4650 2500 50  0000 C CNN
 	1    4650 2500
 	1    0    0    -1
 $EndComp
-Wire Wire Line
-	7350 5100 7350 4950
-Wire Wire Line
-	7350 2950 7350 2200
-Wire Wire Line
-	7850 4250 8050 4250
-Wire Wire Line
-	7850 4350 8050 4350
-Wire Wire Line
-	8050 3150 7850 3150
-Wire Wire Line
-	4450 2900 4450 2700
-Wire Wire Line
-	4550 2700 4550 2900
-Wire Wire Line
-	4650 2700 4650 2900
-Wire Wire Line
-	4750 2700 4750 2900
-Wire Wire Line
-	6550 3100 6550 3150
-Wire Wire Line
-	6550 3150 6850 3150
-Wire Wire Line
-	6450 3100 6450 3250
-Wire Wire Line
-	6450 3250 6850 3250
-Wire Wire Line
-	6350 3100 6350 3350
-Wire Wire Line
-	6350 3350 6850 3350
-Wire Wire Line
-	6250 3100 6250 3450
-Wire Wire Line
-	6250 3450 6850 3450
-Wire Wire Line
-	5950 3100 5950 3550
-Wire Wire Line
-	5950 3550 6850 3550
-Wire Wire Line
-	5850 3100 5850 3650
-Wire Wire Line
-	5850 3650 6850 3650
-Wire Wire Line
-	5750 3100 5750 3750
-Wire Wire Line
-	5750 3750 6850 3750
-Wire Wire Line
-	5650 3100 5650 3850
-Wire Wire Line
-	5650 3850 6850 3850
-Wire Wire Line
-	5350 3100 5350 4050
-Wire Wire Line
-	5350 4050 6850 4050
-Wire Wire Line
-	5250 3100 5250 4150
-Wire Wire Line
-	5250 4150 6850 4150
-Wire Wire Line
-	5150 3100 5150 4250
-Wire Wire Line
-	5150 4250 6850 4250
-Wire Wire Line
-	5050 3100 5050 4350
-Wire Wire Line
-	5050 4350 6850 4350
-Wire Wire Line
-	4750 3100 4750 4450
-Wire Wire Line
-	4750 4450 6850 4450
-Wire Wire Line
-	4650 3100 4650 4550
-Wire Wire Line
-	4650 4550 6850 4550
-Wire Wire Line
-	4550 3100 4550 4650
-Wire Wire Line
-	4550 4650 6850 4650
-Wire Wire Line
-	4450 3100 4450 4750
-Wire Wire Line
-	4450 4750 6850 4750
-Wire Wire Line
-	8100 5100 8100 5000
-Wire Wire Line
-	8100 4800 8100 4700
-Wire Wire Line
-	7850 4550 7900 4550
-Wire Wire Line
-	7900 4550 7900 5100
-Wire Wire Line
-	7850 4650 7900 4650
-Connection ~ 7900 4650
-Wire Wire Line
-	7850 4750 7900 4750
-Connection ~ 7900 4750
-Wire Wire Line
-	4450 2200 4450 2300
-Wire Wire Line
-	4450 2250 4750 2250
-Wire Wire Line
-	4750 2250 4750 2300
-Connection ~ 4450 2250
-Wire Wire Line
-	4650 2250 4650 2300
-Connection ~ 4650 2250
-Wire Wire Line
-	4550 2250 4550 2300
-Connection ~ 4550 2250
 $Comp
 L LED_Small LED4
@@
 F 0 "RN2" V 4950 2500 50  0000 C CNN
 F 1 "330" V 5450 2500 50  0000 C CNN
-F 2 "Resistors_SMD:R_Array_Convex_4x0603" V 5525 2500 50  0001 C CNN
+F 2 "Resistors_SMD:R_Array_Convex_4x0603_HandSoldering" V 5525 2500 50  0001 C CNN
 F 3 "" H 5250 2500 50  0000 C CNN
 	1    5250 2500
 	1    0    0    -1
 $EndComp
-Wire Wire Line
-	5050 2900 5050 2700
-Wire Wire Line
-	5150 2700 5150 2900
-Wire Wire Line
-	5250 2700 5250 2900
-Wire Wire Line
-	5350 2700 5350 2900
-Wire Wire Line
-	5050 2200 5050 2300
-Wire Wire Line
-	5050 2250 5350 2250
-Wire Wire Line
-	5350 2250 5350 2300
-Connection ~ 5050 2250
-Wire Wire Line
-	5250 2250 5250 2300
-Connection ~ 5250 2250
-Wire Wire Line
-	5150 2250 5150 2300
-Connection ~ 5150 2250
 $Comp
 L LED_Small LED8
@@
 F 0 "RN3" V 5550 2500 50  0000 C CNN
 F 1 "330" V 6050 2500 50  0000 C CNN
-F 2 "Resistors_SMD:R_Array_Convex_4x0603" V 6125 2500 50  0001 C CNN
+F 2 "Resistors_SMD:R_Array_Convex_4x0603_HandSoldering" V 6125 2500 50  0001 C CNN
 F 3 "" H 5850 2500 50  0000 C CNN
 	1    5850 2500
 	1    0    0    -1
 $EndComp
-Wire Wire Line
-	5650 2900 5650 2700
-Wire Wire Line
-	5750 2700 5750 2900
-Wire Wire Line
-	5850 2700 5850 2900
-Wire Wire Line
-	5950 2700 5950 2900
-Wire Wire Line
-	5650 2200 5650 2300
-Wire Wire Line
-	5650 2250 5950 2250
-Wire Wire Line
-	5950 2250 5950 2300
-Connection ~ 5650 2250
-Wire Wire Line
-	5850 2250 5850 2300
-Connection ~ 5850 2250
-Wire Wire Line
-	5750 2250 5750 2300
-Connection ~ 5750 2250
 $Comp
 L LED_Small LED12
@@
 F 0 "RN4" V 6150 2500 50  0000 C CNN
 F 1 "330" V 6650 2500 50  0000 C CNN
-F 2 "Resistors_SMD:R_Array_Convex_4x0603" V 6725 2500 50  0001 C CNN
+F 2 "Resistors_SMD:R_Array_Convex_4x0603_HandSoldering" V 6725 2500 50  0001 C CNN
 F 3 "" H 6450 2500 50  0000 C CNN
 	1    6450 2500
 	1    0    0    -1
 $EndComp
-Wire Wire Line
-	6250 2900 6250 2700
-Wire Wire Line
-	6350 2700 6350 2900
-Wire Wire Line
-	6450 2700 6450 2900
-Wire Wire Line
-	6550 2700 6550 2900
-Wire Wire Line
-	6250 2200 6250 2300
-Wire Wire Line
-	6250 2250 6550 2250
-Wire Wire Line
-	6550 2250 6550 2300
-Connection ~ 6250 2250
-Wire Wire Line
-	6450 2250 6450 2300
-Connection ~ 6450 2250
-Wire Wire Line
-	6350 2250 6350 2300
-Connection ~ 6350 2250
 $Comp
 L LED_Small LED16
@@
 	0    -1   -1   0
 $EndComp
+NoConn ~ 7850 3550
+NoConn ~ 7850 3650
+NoConn ~ 6500 2550
+Wire Wire Line
+	7350 5100 7350 4950
+Wire Wire Line
+	7350 2950 7350 2200
+Wire Wire Line
+	7850 4250 8050 4250
+Wire Wire Line
+	7850 4350 8050 4350
+Wire Wire Line
+	8050 3150 7850 3150
+Wire Wire Line
+	4450 2900 4450 2700
+Wire Wire Line
+	4550 2700 4550 2900
+Wire Wire Line
+	4650 2700 4650 2900
+Wire Wire Line
+	4750 2700 4750 2900
+Wire Wire Line
+	8100 5100 8100 5000
+Wire Wire Line
+	8100 4800 8100 4700
+Wire Wire Line
+	7850 4550 7900 4550
+Wire Wire Line
+	7900 4550 7900 5100
+Wire Wire Line
+	7850 4650 7900 4650
+Connection ~ 7900 4650
+Wire Wire Line
+	7850 4750 7900 4750
+Connection ~ 7900 4750
+Wire Wire Line
+	4450 2200 4450 2300
+Wire Wire Line
+	4450 2250 4750 2250
+Wire Wire Line
+	4750 2250 4750 2300
+Connection ~ 4450 2250
+Wire Wire Line
+	4650 2250 4650 2300
+Connection ~ 4650 2250
+Wire Wire Line
+	4550 2250 4550 2300
+Connection ~ 4550 2250
+Wire Wire Line
+	5050 2900 5050 2700
+Wire Wire Line
+	5150 2700 5150 2900
+Wire Wire Line
+	5250 2700 5250 2900
+Wire Wire Line
+	5350 2700 5350 2900
+Wire Wire Line
+	5050 2200 5050 2300
+Wire Wire Line
+	5050 2250 5350 2250
+Wire Wire Line
+	5350 2250 5350 2300
+Connection ~ 5050 2250
+Wire Wire Line
+	5250 2250 5250 2300
+Connection ~ 5250 2250
+Wire Wire Line
+	5150 2250 5150 2300
+Connection ~ 5150 2250
+Wire Wire Line
+	5650 2900 5650 2700
+Wire Wire Line
+	5750 2700 5750 2900
+Wire Wire Line
+	5850 2700 5850 2900
+Wire Wire Line
+	5950 2700 5950 2900
+Wire Wire Line
+	5650 2200 5650 2300
+Wire Wire Line
+	5650 2250 5950 2250
+Wire Wire Line
+	5950 2250 5950 2300
+Connection ~ 5650 2250
+Wire Wire Line
+	5850 2250 5850 2300
+Connection ~ 5850 2250
+Wire Wire Line
+	5750 2250 5750 2300
+Connection ~ 5750 2250
+Wire Wire Line
+	6250 2900 6250 2700
+Wire Wire Line
+	6350 2700 6350 2900
+Wire Wire Line
+	6450 2700 6450 2900
+Wire Wire Line
+	6550 2700 6550 2900
+Wire Wire Line
+	6250 2200 6250 2300
+Wire Wire Line
+	6250 2250 6550 2250
+Wire Wire Line
+	6550 2250 6550 2300
+Connection ~ 6250 2250
+Wire Wire Line
+	6450 2250 6450 2300
+Connection ~ 6450 2250
+Wire Wire Line
+	6350 2250 6350 2300
+Connection ~ 6350 2250
+Wire Wire Line
+	5650 3850 6850 3850
+Wire Wire Line
+	5650 3100 5650 3850
+Wire Wire Line
+	5750 3750 6850 3750
+Wire Wire Line
+	5750 3100 5750 3750
+Wire Wire Line
+	5850 3650 6850 3650
+Wire Wire Line
+	5850 3100 5850 3650
+Wire Wire Line
+	5950 3550 6850 3550
+Wire Wire Line
+	5950 3100 5950 3550
+Wire Wire Line
+	6250 3450 6850 3450
+Wire Wire Line
+	6250 3100 6250 3450
+Wire Wire Line
+	6350 3350 6850 3350
+Wire Wire Line
+	6350 3100 6350 3350
+Wire Wire Line
+	6450 3250 6850 3250
+Wire Wire Line
+	6450 3100 6450 3250
+Wire Wire Line
+	6550 3150 6850 3150
+Wire Wire Line
+	6550 3100 6550 3150
+Wire Wire Line
+	6850 4050 4450 4050
+Wire Wire Line
+	4450 4050 4450 3100
+Wire Wire Line
+	4550 3100 4550 4150
+Wire Wire Line
+	4550 4150 6850 4150
+Wire Wire Line
+	6850 4250 4650 4250
+Wire Wire Line
+	4650 4250 4650 3100
+Wire Wire Line
+	4750 3100 4750 4350
+Wire Wire Line
+	4750 4350 6850 4350
+Wire Wire Line
+	6850 4450 5050 4450
+Wire Wire Line
+	5050 4450 5050 3100
+Wire Wire Line
+	5150 3100 5150 4550
+Wire Wire Line
+	5150 4550 6850 4550
+Wire Wire Line
+	6850 4650 5250 4650
+Wire Wire Line
+	5250 4650 5250 3100
+Wire Wire Line
+	5350 3100 5350 4750
+Wire Wire Line
+	5350 4750 6850 4750
 $EndSCHEMATC

Commit message: hardware/kicad/stm32f030: adding eeprom step1
Parts:
- RN1, RN2, RN3, RN4: value 330 -> 220
Connections:
- net +5V renamed +3V3
- no-connect marks 3 -> 4
Changed lines of the file:
@@
 $Descr A4 11693 8268
 encoding utf-8
-Sheet 4 5
+Sheet 4 6
 Title ""
 Date ""
@@
 sda
 $Comp
-L GND #PWR032
+L GND #PWR38
 U 1 1 58852075
 P 7350 5100
-F 0 "#PWR032" H 7350 4850 50  0001 C CNN
+F 0 "#PWR38" H 7350 4850 50  0001 C CNN
 F 1 "GND" H 7350 4950 50  0000 C CNN
 F 2 "" H 7350 5100 50  0000 C CNN
 F 3 "" H 7350 5100 50  0000 C CNN
 	1    7350 5100
-	1    0    0    -1
-$EndComp
-$Comp
-L +5V #PWR033
-U 1 1 58852090
-P 7350 2200
-F 0 "#PWR033" H 7350 2050 50  0001 C CNN
-F 1 "+5V" H 7350 2340 50  0000 C CNN
-F 2 "" H 7350 2200 50  0000 C CNN
-F 3 "" H 7350 2200 50  0000 C CNN
-	1    7350 2200
 	1    0    0    -1
 $EndComp
@@
 $EndComp
 $Comp
-L GND #PWR034
+L GND #PWR40
 U 1 1 58854DF6
 P 8100 5100
-F 0 "#PWR034" H 8100 4850 50  0001 C CNN
+F 0 "#PWR40" H 8100 4850 50  0001 C CNN
 F 1 "GND" H 8100 4950 50  0000 C CNN
 F 2 "" H 8100 5100 50  0000 C CNN
 F 3 "" H 8100 5100 50  0000 C CNN
 	1    8100 5100
-	1    0    0    -1
-$EndComp
-$Comp
-L +5V #PWR035
-U 1 1 58854E40
-P 8100 4700
-F 0 "#PWR035" H 8100 4550 50  0001 C CNN
-F 1 "+5V" H 8100 4840 50  0000 C CNN
-F 2 "" H 8100 4700 50  0000 C CNN
-F 3 "" H 8100 4700 50  0000 C CNN
-	1    8100 4700
 	1    0    0    -1
 $EndComp
@@
 $EndComp
 $Comp
-L +5V #PWR036
-U 1 1 58854FC3
-P 4450 2200
-F 0 "#PWR036" H 4450 2050 50  0001 C CNN
-F 1 "+5V" H 4450 2340 50  0000 C CNN
-F 2 "" H 4450 2200 50  0000 C CNN
-F 3 "" H 4450 2200 50  0000 C CNN
-	1    4450 2200
-	1    0    0    -1
-$EndComp
-$Comp
-L GND #PWR037
+L GND #PWR39
 U 1 1 58856139
 P 7900 5100
-F 0 "#PWR037" H 7900 4850 50  0001 C CNN
+F 0 "#PWR39" H 7900 4850 50  0001 C CNN
 F 1 "GND" H 7900 4950 50  0000 C CNN
 F 2 "" H 7900 5100 50  0000 C CNN
@@
 P 4650 2500
 F 0 "RN1" V 4350 2500 50  0000 C CNN
-F 1 "330" V 4850 2500 50  0000 C CNN
+F 1 "220" V 4850 2500 50  0000 C CNN
 F 2 "Resistors_SMD:R_Array_Convex_4x0603_HandSoldering" V 4925 2500 50  0001 C CNN
 F 3 "" H 4650 2500 50  0000 C CNN
@@
 $EndComp
 $Comp
-L +5V #PWR038
-U 1 1 588571E4
-P 5050 2200
-F 0 "#PWR038" H 5050 2050 50  0001 C CNN
-F 1 "+5V" H 5050 2340 50  0000 C CNN
-F 2 "" H 5050 2200 50  0000 C CNN
-F 3 "" H 5050 2200 50  0000 C CNN
-	1    5050 2200
-	1    0    0    -1
-$EndComp
-$Comp
 L R_Pack04 RN2
 U 1 1 588571EA
 P 5250 2500
 F 0 "RN2" V 4950 2500 50  0000 C CNN
-F 1 "330" V 5450 2500 50  0000 C CNN
+F 1 "220" V 5450 2500 50  0000 C CNN
 F 2 "Resistors_SMD:R_Array_Convex_4x0603_HandSoldering" V 5525 2500 50  0001 C CNN
 F 3 "" H 5250 2500 50  0000 C CNN
@@
 $EndComp
 $Comp
-L +5V #PWR039
-U 1 1 588572D0
-P 5650 2200
-F 0 "#PWR039" H 5650 2050 50  0001 C CNN
-F 1 "+5V" H 5650 2340 50  0000 C CNN
-F 2 "" H 5650 2200 50  0000 C CNN
-F 3 "" H 5650 2200 50  0000 C CNN
-	1    5650 2200
-	1    0    0    -1
-$EndComp
-$Comp
 L R_Pack04 RN3
 U 1 1 588572D6
 P 5850 2500
 F 0 "RN3" V 5550 2500 50  0000 C CNN
-F 1 "330" V 6050 2500 50  0000 C CNN
+F 1 "220" V 6050 2500 50  0000 C CNN
 F 2 "Resistors_SMD:R_Array_Convex_4x0603_HandSoldering" V 6125 2500 50  0001 C CNN
 F 3 "" H 5850 2500 50  0000 C CNN
@@
 $EndComp
 $Comp
-L +5V #PWR040
-U 1 1 588573D0
-P 6250 2200
-F 0 "#PWR040" H 6250 2050 50  0001 C CNN
-F 1 "+5V" H 6250 2340 50  0000 C CNN
-F 2 "" H 6250 2200 50  0000 C CNN
-F 3 "" H 6250 2200 50  0000 C CNN
-	1    6250 2200
-	1    0    0    -1
-$EndComp
-$Comp
 L R_Pack04 RN4
 U 1 1 588573D6
 P 6450 2500
 F 0 "RN4" V 6150 2500 50  0000 C CNN
-F 1 "330" V 6650 2500 50  0000 C CNN
+F 1 "220" V 6650 2500 50  0000 C CNN
 F 2 "Resistors_SMD:R_Array_Convex_4x0603_HandSoldering" V 6725 2500 50  0001 C CNN
 F 3 "" H 6450 2500 50  0000 C CNN
@@
 Wire Wire Line
 	5350 4750 6850 4750
+NoConn ~ 5900 2500
+$Comp
+L +3.3V #PWR36
+U 1 1 589C0D19
+P 7350 2200
+F 0 "#PWR36" H 7350 2050 50  0001 C CNN
+F 1 "+3.3V" H 7350 2340 50  0000 C CNN
+F 2 "" H 7350 2200 50  0000 C CNN
+F 3 "" H 7350 2200 50  0000 C CNN
+	1    7350 2200
+	1    0    0    -1
+$EndComp
+$Comp
+L +3.3V #PWR37
+U 1 1 589C10A0
+P 8100 4700
+F 0 "#PWR37" H 8100 4550 50  0001 C CNN
+F 1 "+3.3V" H 8100 4840 50  0000 C CNN
+F 2 "" H 8100 4700 50  0000 C CNN
+F 3 "" H 8100 4700 50  0000 C CNN
+	1    8100 4700
+	1    0    0    -1
+$EndComp
+$Comp
+L +3.3V #PWR35
+U 1 1 589C18FA
+P 6250 2200
+F 0 "#PWR35" H 6250 2050 50  0001 C CNN
+F 1 "+3.3V" H 6250 2340 50  0000 C CNN
+F 2 "" H 6250 2200 50  0000 C CNN
+F 3 "" H 6250 2200 50  0000 C CNN
+	1    6250 2200
+	1    0    0    -1
+$EndComp
+$Comp
+L +3.3V #PWR34
+U 1 1 589C1947
+P 5650 2200
+F 0 "#PWR34" H 5650 2050 50  0001 C CNN
+F 1 "+3.3V" H 5650 2340 50  0000 C CNN
+F 2 "" H 5650 2200 50  0000 C CNN
+F 3 "" H 5650 2200 50  0000 C CNN
+	1    5650 2200
+	1    0    0    -1
+$EndComp
+$Comp
+L +3.3V #PWR33
+U 1 1 589C1994
+P 5050 2200
+F 0 "#PWR33" H 5050 2050 50  0001 C CNN
+F 1 "+3.3V" H 5050 2340 50  0000 C CNN
+F 2 "" H 5050 2200 50  0000 C CNN
+F 3 "" H 5050 2200 50  0000 C CNN
+	1    5050 2200
+	1    0    0    -1
+$EndComp
+$Comp
+L +3.3V #PWR32
+U 1 1 589C19E1
+P 4450 2200
+F 0 "#PWR32" H 4450 2050 50  0001 C CNN
+F 1 "+3.3V" H 4450 2340 50  0000 C CNN
+F 2 "" H 4450 2200 50  0000 C CNN
+F 3 "" H 4450 2200 50  0000 C CNN
+	1    4450 2200
+	1    0    0    -1
+$EndComp
 $EndSCHEMATC
